File: clickwheel_breakout_4th_gen.kicad_pcb (KiCad board)
At the start: 2 copper layers, 55.5 x 98.2 mm, 8 parts, among them J1 SFV8R-2STE1HLF, J2 SFV14R-2STE1HLF, J3 SFV8R-2STE1HLF, J4 SFV14R-2STE1HLF, J5 Conn_02x08_Odd_Even, J6 Conn_02x14_Odd_Even, J7 USB_C_Receptacle_USB2.0

Commit message: fix qr code name
Parts:
- QR1: footprint clickwheel_breakout_4th_gen-qr:QR_data -> QR:QR_data
- moved QR1 0.75 mm to (62.4, 66.5)

Commit message: ci: move qr code to front for now (INTI-CMNB/KiBot#271)
Parts:
- QR1: moved to F.Cu
- moved QR1 5.46 mm to (61.8, 71.9), turned to 0 degrees
