File: clickwheel_breakout_4th_gen.kicad_pcb (KiCad board)
At the start: 2 copper layers, 55.5 x 98.2 mm, 8 parts, among them J1 SFV8R-2STE1HLF, J2 SFV14R-2STE1HLF, J3 SFV8R-2STE1HLF, J4 SFV14R-2STE1HLF, J5 Conn_02x08_Odd_Even, J6 Conn_02x14_Odd_Even, J7 USB_C_Receptacle_USB2.0

Commit message: project: update to kicad 7, remove qr code
Parts:
- removed QR1: QR_data, QR:QR_data

Commit message: feature: update revision info
Other:
- board text added: "1"
- board text added: "10"
- board text added: "11"
- board text added: "12"
- board text added: "13"
- board text added: "14"
- board text added: "2"
- board text added: "3"
- board text added: "4"
- board text added: "5"
- board text added: "6"
- board text added: "7"
- board text added: "8"
- board text added: "9"
- board text added: "BTN1"
- board text added: "CFG1"
- board text added: "SCK"
- board text added: "iPod Photo Breakout ${TAG} (${HASH}) ${DATE}"
- board text removed: "EN2"
- board text removed: "SCL"
- board text removed: "iPod Photo Breakout Rev 1"
Changed lines of the file:
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@@
   )
   (property "DATE" "YYYY-MM-DD HH:MM:SS")
-  (property "REVISION" "DEV")
+  (property "HASH" "deadbeef")
+  (property "TAG" "TAG")
   (net 0 "")
   (net 1 "unconnected-(J1-PadM2)")
@@
     )
   )
-  (gr_line (start 72.136 70.612) (end 70.104 70.612)
+  (gr_line (start 71.1454 70.612) (end 70.104 70.612)
     (stroke (width 0.12) (type solid)) (layer "F.SilkS"))
   (gr_line (start 70.104 70.612) (end 70.104 74.422)
@@
   (gr_line (start 70.104 80.772) (end 70.104 76.708)
     (stroke (width 0.12) (type solid)) (layer "F.SilkS"))
-  (gr_line (start 72.136 80.772) (end 70.104 80.772)
+  (gr_line (start 71.1454 80.772) (end 70.104 80.772)
     (stroke (width 0.12) (type solid)) (layer "F.SilkS"))
   (gr_arc (start 69.596 75.184) (mid 69.909597 74.714669) (end 70.46321 74.82479)
@@
     (effects (font (size 1 1) (thickness 0.15)) (justify mirror))
   )
-  (gr_text "EN1" (at 47.244 70.358) (layer "F.SilkS")
-    (effects (font (size 1 1) (thickness 0.15)) (justify right))
-  )
-  (gr_text "VBAT" (at 47.244 85.598) (layer "F.SilkS")
-    (effects (font (size 1 1) (thickness 0.15)) (justify right))
-  )
-  (gr_text "SCL" (at 47.244 83.058) (layer "F.SilkS")
-    (effects (font (size 1 1) (thickness 0.15)) (justify right))
-  )
-  (gr_text "EN2" (at 47.244 80.518) (layer "F.SilkS")
-    (effects (font (size 1 1) (thickness 0.15)) (justify right))
-  )
-  (gr_text "SDA" (at 47.244 72.898) (layer "F.SilkS")
-    (effects (font (size 1 1) (thickness 0.15)) (justify right))
-  )
-  (gr_text "GND" (at 47.244 67.818) (layer "F.SilkS")
+  (gr_text "EN1" (at 47.6758 70.358) (layer "F.SilkS")
+    (effects (font (size 1 1) (thickness 0.15)) (justify right))
+  )
+  (gr_text "VBAT" (at 47.6758 85.598) (layer "F.SilkS")
+    (effects (font (size 1 1) (thickness 0.15)) (justify right))
+  )
+  (gr_text "SCK" (at 47.6758 83.058) (layer "F.SilkS")
+    (effects (font (size 1 1) (thickness 0.15)) (justify right))
+  )
+  (gr_text "CFG1" (at 47.6758 80.518) (layer "F.SilkS")
+    (effects (font (size 1 1) (thickness 0.15)) (justify right))
+  )
+  (gr_text "SDA" (at 47.6758 72.898) (layer "F.SilkS")
+    (effects (font (size 1 1) (thickness 0.15)) (justify right))
+  )
+  (gr_text "GND" (at 47.6758 67.818) (layer "F.SilkS")
     (effects (font (size 1 1) (thickness 0.15)) (justify right))
   )
@@
     (effects (font (size 1 1) (thickness 0.15)) (justify left))
   )
+  (gr_text "4" (at 53.086 77.978) (layer "F.SilkS")
+    (effects (font (size 1 1) (thickness 0.15)) (justify left))
+  )
   (gr_text "Connect to\nheadphone\nboard" (at 94.25 58.55) (layer "F.SilkS")
     (effects (font (size 1 1) (thickness 0.15)) (justify right))
@@
     (effects (font (size 1 1) (thickness 0.15)) (justify left))
   )
+  (gr_text "8" (at 53.086 67.818) (layer "F.SilkS")
+    (effects (font (size 1 1) (thickness 0.15)) (justify left))
+  )
+  (gr_text "1" (at 72.2376 88.392) (layer "F.SilkS")
+    (effects (font (size 1 1) (thickness 0.15)) (justify right))
+  )
+  (gr_text "7" (at 53.086 70.358) (layer "F.SilkS")
+    (effects (font (size 1 1) (thickness 0.15)) (justify left))
+  )
   (gr_text "HPSL_VIDEO" (at 77.724 68.072) (layer "F.SilkS")
     (effects (font (size 1 1) (thickness 0.15)) (justify left))
   )
+  (gr_text "2" (at 72.2376 85.852) (layer "F.SilkS")
+    (effects (font (size 1 1) (thickness 0.15)) (justify right))
+  )
+  (gr_text "1" (at 53.086 85.598) (layer "F.SilkS")
+    (effects (font (size 1 1) (thickness 0.15)) (justify left))
+  )
+  (gr_text "5" (at 53.086 75.438) (layer "F.SilkS")
+    (effects (font (size 1 1) (thickness 0.15)) (justify left))
+  )
   (gr_text "RMT3_DGND" (at 77.724 70.612) (layer "F.SilkS")
     (effects (font (size 1 1) (thickness 0.15)) (justify left))
   )
+  (gr_text "13" (at 72.2376 57.912) (layer "F.SilkS")
+    (effects (font (size 1 1) (thickness 0.15)) (justify right))
+  )
+  (gr_text "3" (at 72.2376 83.312) (layer "F.SilkS")
+    (effects (font (size 1 1) (thickness 0.15)) (justify right))
+  )
+  (gr_text "9" (at 72.2376 68.072) (layer "F.SilkS")
+    (effects (font (size 1 1) (thickness 0.15)) (justify right))
+  )
+  (gr_text "10" (at 72.2376 65.532) (layer "F.SilkS")
+    (effects (font (size 1 1) (thickness 0.15)) (justify right))
+  )
   (gr_text "RMT2_TxD" (at 77.724 60.452) (layer "F.SilkS")
     (effects (font (size 1 1) (thickness 0.15)) (justify left))
   )
+  (gr_text "11" (at 72.2376 62.992) (layer "F.SilkS")
+    (effects (font (size 1 1) (thickness 0.15)) (justify right))
+  )
   (gr_text "SHIELD1" (at 77.724 55.372) (layer "F.SilkS")
     (effects (font (size 1 1) (thickness 0.15)) (justify left))
   )
+  (gr_text "3" (at 53.086 80.518) (layer "F.SilkS")
+    (effects (font (size 1 1) (thickness 0.15)) (justify left))
+  )
   (gr_text "Headphone\npassthrough\nto mainboard" (at 55.1 60.3) (layer "F.SilkS")
     (effects (font (size 1 1) (thickness 0.15)) (justify right))
   )
-  (gr_text "iPod Photo Breakout Rev 1\n" (at 41.91 109.855 90) (layer "F.SilkS")
-    (effects (font (size 1.5 1.5) (thickness 0.3)))
+  (gr_text "BTN1" (at 47.6758 78.008) (layer "F.SilkS")
+    (effects (font (size 1 1) (thickness 0.15)) (justify right))
+  )
+  (gr_text "12" (at 72.2376 60.452) (layer "F.SilkS")
+    (effects (font (size 1 1) (thickness 0.15)) (justify right))
+  )
+  (gr_text "4" (at 72.2376 80.772) (layer "F.SilkS")
+    (effects (font (size 1 1) (thickness 0.15)) (justify right))
+  )
+  (gr_text "14" (at 72.2376 55.372) (layer "F.SilkS")
+    (effects (font (size 1 1) (thickness 0.15)) (justify right))
+  )
+  (gr_text "5" (at 72.2376 78.232) (layer "F.SilkS")
+    (effects (font (size 1 1) (thickness 0.15)) (justify right))
   )
   (gr_text "RMT1_RxD" (at 77.724 57.912) (layer "F.SilkS")
@@
     (effects (font (size 1 1) (thickness 0.15)) (justify left))
   )
+  (gr_text "7" (at 72.2376 73.152) (layer "F.SilkS")
+    (effects (font (size 1 1) (thickness 0.15)) (justify right))
+  )
+  (gr_text "8" (at 72.2376 70.612) (layer "F.SilkS")
+    (effects (font (size 1 1) (thickness 0.15)) (justify right))
+  )
+  (gr_text "6" (at 72.2376 75.692) (layer "F.SilkS")
+    (effects (font (size 1 1) (thickness 0.15)) (justify right))
+  )
   (gr_text "HPR1_R" (at 77.724 75.692) (layer "F.SilkS")
     (effects (font (size 1 1) (thickness 0.15)) (justify left))
   )
+  (gr_text "6" (at 53.086 72.898) (layer "F.SilkS")
+    (effects (font (size 1 1) (thickness 0.15)) (justify left))
+  )
+  (gr_text "2" (at 53.086 83.058) (layer "F.SilkS")
+    (effects (font (size 1 1) (thickness 0.15)) (justify left))
+  )
+  (gr_text "iPod Photo Breakout\n${TAG}\n(${HASH})\n${DATE}" (at 51.7 53.5) (layer "F.Mask")
+    (effects (font (size 1 1) (thickness 0.15)) (justify bottom))
+  )
   (gr_text "Connect LCK_COM to DGND to unlock controls" (at 96.774 80.772) (layer "Cmts.User")
