File: clickwheel_breakout_4th_gen.kicad_sch (KiCad schematic)
At the start: 8 parts, among them J1 SFV8R-2STE1HLF, J2 SFV14R-2STE1HLF, J3 SFV8R-2STE1HLF, J4 SFV14R-2STE1HLF, J5 Conn_02x08_Odd_Even, J6 Conn_02x14_Odd_Even, J7 USB_C_Receptacle_USB2.0

Commit message: ci: export schematics
Other:
- title: (none) -> iPod 4th Gen Clickwheel Breakout
Changed lines of the file:
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@@
 (kicad_sch (version 20211123) (generator eeschema)
   (paper "A4")
+  (title_block
+    (title "iPod 4th Gen Clickwheel Breakout")
+    (date "${DATE}")
+    (rev "${REVISION}")
+  )
   (no_connect (at 78.74 77.47))
   (no_connect (at 78.74 80.01))
